File: KiCAD/Nabu_MEGAMAPPER/_autosave-Nabu_MEGAMAPPER.kicad_pcb (KiCad board)
At the start: 2 copper layers, 41 parts, among them J1 Z80 Socket Header, J2 Z80 Socket Header, J3 JTAG, U1 Z80CPU, U10 74LS374, U11 74LS374, U12 74LS85, U13 XC9536PC44, U14 74LS139, U15 AS6C4008-55PCN, U16 AS6C4008-55PCN, U17 AS6C4008-55PCN, U18 AS6C4008-55PCN, U19 74LS245, U2 74LS32, U3 74LS670, U4 74LS670, U5 HM6116, U6 74LS157, U7 74LS157, U8 74LS157, U9 74LS244

Commit message: Started laying out MegaMapper PCB
Parts:
- moved U3 353.0 mm to (233.7, 78.7)
- moved U4 322.9 mm to (214.6, 69.2)
- moved C3 288.9 mm to (240.0, 75.5), turned to 180 degrees
- moved C4 271.3 mm to (220.9, 66.0), turned to 180 degrees
- moved U15 268.8 mm to (139.7, 97.8)
- moved U19 255.8 mm to (186.7, 111.1)
- moved U12 246.7 mm to (180.3, 94.6), turned to 90 degrees
- moved U11 242.8 mm to (162.6, 64.8)
- moved U10 239.7 mm to (148.6, 64.8)
- moved U9 236.6 mm to (134.6, 64.8)
- moved U16 230.6 mm to (118.1, 97.8)
- moved C19 219.8 mm to (188.0, 107.9)
- moved C1 214.5 mm to (166.4, 94.6)
- moved C11 212.6 mm to (168.9, 61.6), turned to 180 degrees
- moved C10 198.1 mm to (154.9, 61.6), turned to 180 degrees
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